Commit message: added environment (Europalette); added node to show EPAL in Rviz not in gazebo; changed launchfiles accordingly; Robots now connected to world

File: src/environment/urdf/Europalette.urdf (robot description, URDF)
Before this commit: robot Europalette, 1 links, 0 joints
Links:
- added link world
- link base_link: geometry collision mesh filename=package://environment/meshes/Europoolpalette_scaled.stl; visual mesh filename=package://environment/meshes/Europoolpalette_scaled.stl
Joints:
- added joint europalette_to_world: type floating, parent world, child base_link, origin xyz=-2 -2 0.1 rpy=0 0 0

Commit message: robAssemble is fixed

File: src/environment/urdf/Europalette.urdf (robot description, URDF)
Before this commit: robot europalette, 2 links, 1 joints
Links:
- removed link world
Joints:
- removed joint europalette_to_world

File: src/project_assem/urdf/RobAssemble.urdf (robot description, URDF)
Before this commit: robot rob_assemble, 6 links, 5 joints
Links:
- removed link Glied1
- removed link Glied2
- removed link Glied3
- removed link Glied4
- added link Endeffektor, mass 0.0538557572339802; collision mesh filename=package://project_assem/meshes/Endeffektor.STL; visual mesh filename=package://project_assem/meshes/Endeffektor.STL
- added link Link1, mass 8.06345148807657; collision mesh filename=package://project_assem/meshes/Link1_2.STL; visual mesh filename=package://project_assem/meshes/Link1_2.STL
- added link Link2, mass 7.6161855101175; collision mesh filename=package://project_assem/meshes/Link2_3.STL; visual mesh filename=package://project_assem/meshes/Link2_3.STL
- added link Link3, mass 4.610306124135; collision mesh filename=package://project_assem/meshes/Link3_5.STL; visual mesh filename=package://project_assem/meshes/Link3_5.STL
- added link Link4, mass 1.02538578363401; collision mesh filename=package://project_assem/meshes/Link4.STL; visual mesh filename=package://project_assem/meshes/Link4.STL
- added link Link5, mass 1.55208868418314; collision mesh filename=package://project_assem/meshes/Link5.STL; visual mesh filename=package://project_assem/meshes/Link5.STL
- link base_link: geometry collision mesh filename=package://project_assem/meshes/base_link_2.STL; visual mesh filename=package://project_assem/meshes/base_link_2.STL
Joints:
- added joint Endeffektor_Joint: type continuous, parent Link5, child Endeffektor, origin xyz=0 0 0.215 rpy=0 3.14159 0, axis 0 0 1
- added joint Joint5: type continuous, parent Link4, child Link5, origin xyz=0.00008 -0.00005 0.2068 rpy=0 0 0, axis 0 0 1, limit lower=-1 upper=1 effort=100 velocity=0.1
- joint Joint1: child Glied1 -> Link1; origin xyz=-0.019125 -0.35586 0.21258 rpy=-1.5708 -0.17308 3.1416 -> xyz=0 0 0.155 rpy=0 0 0
- joint Joint2: child Glied2 -> Link2; origin xyz=0 -0.061397 0.16273 rpy=3.1416 -1.0187 -3.1416 -> xyz=0 -0.02 0.1628 rpy=0 0 0; parent Glied1 -> Link1
- joint Joint3: child Glied3 -> Link3; origin xyz=0.585 0.033821 0 rpy=3.1416 0.62131 3.1416 -> xyz=0.585149 -0.09 0.000162 rpy=3.14159 0 3.14159; parent Glied2 -> Link2
- joint Joint4: child Glied4 -> Link4; origin xyz=0.64623 0.22735 0 rpy=-2.7786 0 0.017453 -> xyz=0.75 -0.093 0 rpy=0 -1.5708 3.14159; parent Glied3 -> Link3; type revolute -> continuous
- joint base_to_world: origin xyz=2 2 -0.15 rpy=-1.5708 0 0 -> xyz=2 2 0 rpy=0 0 0

Commit message: Alle Teile und Roboter werden basic geladen und angezeigt

File: src/environment/urdf/Europalette.urdf (robot description, URDF)
Before this commit: robot europalette, 1 links, 0 joints
Links:
- link base_link: geometry collision mesh filename=package://environment/meshes/europalette/Europoolpalette_sc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; visual mesh filename=package://environment/meshes/europalette/Europoolpalette_sc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

File: src/environment/urdf/conveyor.urdf (robot description, URDF)
Before this commit: robot conveyor, 2 links, 1 joints
Links:
- added link belt, mass 3.53662299561806; collision mesh filename=package://environment/meshes/conveyor/belt.STL; visual mesh filename=package://environment/meshes/conveyor/belt.STL
- link conveyor_link: mass 3.53662299561806 -> 18.686505647015; geometry collision mesh filename=package://environment/meshes/conveyor/conveyor_link.STL; visual mesh filename=package://environment/meshes/conveyor/conveyor_link.STL
Joints:
- added joint belt: type fixed, parent conveyor_link, child belt, origin xyz=-0.241229392828482 -1.07757386726348 0.401876129111459 rpy=1.5707963267949 0 1.5707963267949, axis 0 0 0
- joint conveyor_to_world: type floating -> fixed
