Commit message: Updated brick spawner; europalette spawns on conveyor; conveyor updated (conveyor gazebo plugin)

File: src/environment/urdf/brick.urdf (robot description, URDF)
Before this commit: robot brick, 2 links, 1 joints
Links:
- removed link world
- link brick: mass 9.7387642147252 -> 6
Joints:
- removed joint brick_to_world

File: src/environment/urdf/conveyor.urdf (robot description, URDF)
Before this commit: robot conveyor, 3 links, 2 joints
Links:
- removed link belt
- removed link conveyor_link
- added link belt_moving, mass 10; collision box size=0.425 1.2 0.001
- added link belt_visual, mass 71.953; collision mesh filename=package://environment/meshes/conveyor/conveyor_belt.stl; visual mesh filename=package://environment/meshes/conveyor/conveyor_belt.stl
Joints:
- removed joint belt
- removed joint conveyor_to_world
- added joint belt_joint: type prismatic, parent belt_visual, child belt_moving, origin xyz=0.0 0.0 0.74 rpy=0.0 0.0 0.0, axis 0 1 0, limit lower=-1 upper=1 effort=100000 velocity=100000
- added joint fixed: type fixed, parent world, child belt_visual, origin xyz=-2 -2 0.0 rpy=0.0 0.0 0
