Commit message: full setup launch file

File: src/environment/urdf/europalette.urdf (robot description, URDF)
Before this commit: robot europalette, 1 links, 0 joints
Links:
- added link world
Joints:
- added joint fixed: type fixed, parent world, child base_link, origin xyz=-2 -2 0.0 rpy=0.0 0.0 0
