Commit message: RobAssemble und RobShift werden beide in gazebo geladen und können grundsätzlich gesteuert werden

File: src/project_assem/urdf/RobAssemble.urdf (robot description, URDF)
Before this commit: robot Assem1, 5 links, 4 joints
Links:
- removed link Glied 1
- removed link glied3
- removed link glied4
- added link Glied1, mass 8.06345148807656; collision mesh filename=package://project_assem/meshes/Glied1.STL; visual mesh filename=package://project_assem/meshes/Glied1.STL
- added link Glied3, mass 4.61023011928217; collision mesh filename=package://project_assem/meshes/Glied3.STL; visual mesh filename=package://project_assem/meshes/Glied3.STL
- added link Glied4, mass 1.77228640360948; collision mesh filename=package://project_assem/meshes/Glied4.STL; visual mesh filename=package://project_assem/meshes/Glied4.STL
- added link world
Joints:
- removed joint joint 1
- removed joint joint 2
- removed joint joint4
- removed joint link3
- added joint Joint1: type continuous, parent base_link, child Glied1, origin xyz=-0.019125 -0.35586 0.21258 rpy=1.5708 1.0635 0, axis 0 0 1
- added joint Joint2: type continuous, parent Glied1, child Glied2, origin xyz=0 0 0.16273 rpy=0 -1.1634 0, axis 0 1 0
- added joint Joint3: type continuous, parent Glied2, child Glied3, origin xyz=0.585 -0.16334 0 rpy=3.1416 1.1417 3.1416, axis 0 1 0
- added joint Joint4: type continuous, parent Glied3, child Glied4, origin xyz=0.68528 0.36379 0 rpy=-0.94737 0 0.017453, axis 1 0 0
- added joint base_to_world: type fixed, parent world, child base_link, origin xyz=7 7 -0.19 rpy=-1.5708 0 0

Commit message: robshift und robAssemble werden in gazebo, rviz geladen. rviz bildet den zustand der roboter aus gazebo ab. Problem: robAssemble springt zwischen seiner initilposition und der aktuellen position

File: src/project_assem/urdf/RobAssemble.urdf (robot description, URDF)
Before this commit: robot rob_assemble, 6 links, 5 joints
Joints:
- joint base_to_world: origin xyz=7 7 -0.19 rpy=-1.5708 0 0 -> xyz=2 2 -0.19 rpy=-1.5708 0 0

Commit message: Roboter werden in Rviz, gazebo geladen und können über das topic gesteuert werden

File: src/project_assem/urdf/RobAssemble.urdf (robot description, URDF)
Before this commit: robot rob_assemble, 6 links, 5 joints
Joints:
- joint base_to_world: origin xyz=2 2 -0.19 rpy=-1.5708 0 0 -> xyz=2 2 -0.15 rpy=-1.5708 0 0

File: src/project_model/urdf/RobShift.urdf (robot description, URDF)
Before this commit: robot project_model, 9 links, 8 joints
Joints:
- joint base_to_world: origin xyz=0 0 0.08 rpy=0 0 0 -> xyz=0 0 0.2 rpy=0 0 0

Commit message: Urdf Robshift und RobAssemble angepasst. Flackern bei RobAssemble korrigiert, Achsen lassen sich bewegen. RobAssemble hat Probleme ab Joint3 folgend, Achsen scheinen nicht zu passen

File: src/project_assem/urdf/RobAssemble.urdf (robot description, URDF)
Before this commit: robot rob_assemble, 6 links, 5 joints
Links:
- link Glied1: mass 8.06345148807656 -> 8.06345148807657
- link Glied2: mass 7.61618558267862 -> 7.61618748268792
- link Glied3: mass 4.61023011928217 -> 4.6103173169206
- link Glied4: mass 1.77228640360948 -> 1.77228640360949
Joints:
- joint Joint1: limit (none) -> lower=-3.2 upper=3.2 effort=1000 velocity=0.5; origin xyz=-0.019125 -0.35586 0.21258 rpy=1.5708 1.0635 0 -> xyz=-0.019125 -0.35586 0.21258 rpy=-1.5708 -0.17308 3.1416; type continuous -> revolute
- joint Joint2: limit (none) -> lower=-1.2 upper=1.2 effort=1000 velocity=0.2; origin xyz=0 0 0.16273 rpy=0 -1.1634 0 -> xyz=0 -0.061397 0.16273 rpy=3.1416 -1.0187 -3.1416; type continuous -> revolute
- joint Joint3: limit (none) -> lower=-3.16 upper=3.16 effort=100 velocity=0.5; origin xyz=0.585 -0.16334 0 rpy=3.1416 1.1417 3.1416 -> xyz=0.585 0.033821 0 rpy=3.1416 0.62131 3.1416; type continuous -> revolute
- joint Joint4: limit (none) -> lower=-10 upper=10 effort=20 velocity=0.2; origin xyz=0.68528 0.36379 0 rpy=-0.94737 0 0.017453 -> xyz=0.64623 0.22735 0 rpy=-2.7786 0 0.017453; type continuous -> revolute

File: src/project_model/urdf/RobShift.urdf (robot description, URDF)
Before this commit: robot project_model, 9 links, 8 joints
Joints:
- joint Endeffektor_Joint: axis 0 0 1 -> 0.18605 0.37106 0.90978; origin xyz=0.215447561272202 -0.128958924945047 -0.0318164852676601 rpy=1.44045339925499 0.872427010505441 -2.82137203630719 -> xyz=0 -0.15357 -0.016296 rpy=1.5708 0.90331 3.1416
- joint Joint2: limit lower=-3.2289 upper=1.1345 effort=1000.0 velocity=0.5 -> lower=-1.0 upper=0.8 effort=1000.0 velocity=0.25; origin xyz=-0.34871 0 0.25746 rpy=1.5708 0.95413 3.1416 -> xyz=-0.34871 0 0.25746 rpy=1.5708 1.077 3.1416
- joint Joint3: limit lower=-3.194 upper=3.0543 effort=1000.0 velocity=0.5 -> lower=-2 upper=2 effort=1000.0 velocity=0.5; origin xyz=-1.20000000000001 0 0.36512066324591 rpy=0 0 -2.50263118864038 -> xyz=-1.2 0 0.36512 rpy=0 0 -2.3798
- joint Joint4: limit lower=-6.10865238198015 upper=6.10865238198015 effort=1000.0 velocity=0.5 -> lower=-1.0 upper=1.0 effort=100.0 velocity=0.1; origin xyz=-1.14996945665964 -0.0398016920240907 0.0752588050980933 rpy=-1.5707963267949 0.495267839274662 1.5707963267949 -> xyz=-1.15 -0.039802 0.075259 rpy=-1.5708 0.49527 1.5708
- joint Joint5: limit lower=-2.0943951023932 upper=2.0943951023932 effort=1000.0 velocity=0.5 -> lower=0 upper=0 effort=1000.0 velocity=0.5; origin xyz=0 0 0.146319270574909 rpy=0 0 -2.99190622753308 -> xyz=0 0 0.14632 rpy=0 0 -2.9919
- joint Joint6: axis 0 0 1 -> -0.068076 -0.12139 0.99027; limit lower=-6.1087 upper=6.1087 effort=1000.0 velocity=0.5 -> lower=0 upper=0 effort=1000.0 velocity=0.5; origin xyz=0.0094648 0.014522 0.24788 rpy=-1.4549 0.92347 2.6583 -> xyz=-0.0088287 -0.013655 0.24866 rpy=-1.6508 0.50975 2.5265

Commit message: RobAssem fixed;

File: src/project_assem/urdf/RobAssemble.urdf (robot description, URDF)
Before this commit: robot rob_assemble, 8 links, 7 joints
Joints:
- joint Endeffektor_Joint: limit (none) -> lower=-1 upper=1 effort=100 velocity=0.1; origin xyz=0 0 0.215 rpy=0 3.14159 0 -> xyz=0 0 0.21 rpy=0 3.14159 0; type continuous -> revolute
- joint Joint4: axis 1 0 0 -> 0 0 1
- joint Joint5: axis 0 0 1 -> 0 1 0

File: src/project_model/urdf/RobShift.urdf (robot description, URDF)
Before this commit: robot project_model, 9 links, 8 joints
Links:
- removed link Endeffektor
- removed link Link5
- removed link Link6
- added link Vakuumgreifer, mass 0.87056; collision mesh filename=package://project_model/meshes/Vakuumgreifer.STL; visual mesh filename=package://project_model/meshes/Vakuumgreifer.STL
- link Link1: mass 85.6566874789417 -> 85.657
- link Link2: mass 51.8329786183893 -> 51.8329784346567
- link Link3: mass 27.6329069261582 -> 27.633
- link Link4: mass 0.850036432245057 -> 1.7447; geometry collision mesh filename=package://project_model/meshes/Link4.STL; visual mesh filename=package://project_model/meshes/Link4.STL
- link base_link: mass 30.1843359271744 -> 30.184
Joints:
- removed joint Endeffektor_Joint
- removed joint Joint5
- removed joint Joint6
- added joint Joint_Vakuumgreifer: type continuous, parent Link4, child Vakuumgreifer, origin xyz=0.28437 0.0023885 0.0039722 rpy=2.4444 -0.63915 0.46331, axis 0 1 0
- joint Joint4: origin xyz=-0.0435 1.275 -0.025 rpy=-1.5708 0 0 -> xyz=-0.0435 1.21 -0.025 rpy=0 0 1.5708

Commit message: Attach Dettach working

File: src/project_assem/urdf/RobAssemble.urdf (robot description, URDF)
Before this commit: robot rob_assemble, 8 links, 7 joints
Joints:
- joint Joint4: type continuous -> revolute
- joint Joint5: type continuous -> revolute
