Commit message: RobShift ist grundlegend beweglich

File: src/project_model/urdf/RobShift.urdf (robot description, URDF)
Before this commit: robot project_model, 8 links, 7 joints
Links:
- added link world
Joints:
- added joint base_to_world: type fixed, parent world, child base_link, origin xyz=0 0 0.08 rpy=0 0 0
- joint Endeffektor_Joint: limit lower=0 upper=0 effort=0 velocity=0 -> lower=0 upper=0 effort=1000.0 velocity=0.5
- joint Joint1: limit lower=-3.1416 upper=3.1416 effort=0 velocity=0 -> lower=-3.1416 upper=3.1416 effort=1000.0 velocity=0.5
- joint Joint2: limit lower=-3.2289 upper=1.1345 effort=0 velocity=0 -> lower=-3.2289 upper=1.1345 effort=1000.0 velocity=0.5
- joint Joint3: limit lower=-3.194 upper=3.0543 effort=0 velocity=0 -> lower=-3.194 upper=3.0543 effort=1000.0 velocity=0.5
- joint Joint4: limit lower=-6.10865238198015 upper=6.10865238198015 effort=0 velocity=0 -> lower=-6.10865238198015 upper=6.10865238198015 effort=1000.0 velocity=0.5
- joint Joint5: limit lower=-2.0943951023932 upper=2.0943951023932 effort=0 velocity=0 -> lower=-2.0943951023932 upper=2.0943951023932 effort=1000.0 velocity=0.5
- joint Joint6: limit lower=-6.1087 upper=6.1087 effort=0 velocity=0 -> lower=-6.1087 upper=6.1087 effort=1000.0 velocity=0.5

Commit message: Fixed robshift: Joint3 und Link3 jetzt connected und funktionsfähig. Controller läuft, muss noch justiert werden.

File: src/project_model/urdf/RobShift.urdf (robot description, URDF)
Before this commit: robot project_model, 9 links, 8 joints
Joints:
- joint Joint3: origin xyz=-1.2 0 0.36512 rpy=0 0 -2.3798 -> xyz=-1.0358 -0.6058 0.465 rpy=0 0 3.14159

Commit message: Robshift funktionsfähig, kann angesteuert werden. Joints und Links verhalten sich jetzt erwartungsgemäß.

File: src/project_model/urdf/RobShift.urdf (robot description, URDF)
Before this commit: robot project_model, 9 links, 8 joints
Links:
- link Link3: geometry collision mesh filename=package://project_model/meshes/Link3_3.STL; visual mesh filename=package://project_model/meshes/Link3_3.STL
- link Link4: geometry collision mesh filename=package://project_model/meshes/Link4_2.STL; visual mesh filename=package://project_model/meshes/Link4_2.STL
- link Link5: geometry collision mesh filename=package://project_model/meshes/Link5_4.STL; visual mesh filename=package://project_model/meshes/Link5_4.STL
- link Link6: geometry collision mesh filename=package://project_model/meshes/Link6_6.STL; visual mesh filename=package://project_model/meshes/Link6_6.STL
Joints:
- joint Joint3: origin xyz=-1.0358 -0.6058 0.465 rpy=0 0 3.14159 -> xyz=-1.0358 -0.6058 0.465 rpy=0 0 0
- joint Joint4: limit lower=-1.0 upper=1.0 effort=100.0 velocity=0.1 -> lower=-3 upper=3 effort=100.0 velocity=0.1; origin xyz=-1.15 -0.039802 0.075259 rpy=-1.5708 0.49527 1.5708 -> xyz=-0.0435 1.275 -0.025 rpy=-1.5708 0 0
- joint Joint5: origin xyz=0 0 0.14632 rpy=0 0 -2.9919 -> xyz=0 0 0 rpy=0 0 0
- joint Joint6: axis -0.068076 -0.12139 0.99027 -> 0 1 0; limit lower=0 upper=0 effort=1000.0 velocity=0.5 -> lower=-2 upper=2 effort=100.0 velocity=0.2; origin xyz=-0.0088287 -0.013655 0.24866 rpy=-1.6508 0.50975 2.5265 -> xyz=0.00008 -0.00005 0.2068 rpy=0 0 0

Commit message: working robo shift with attach dettach

File: src/project_model/urdf/RobShift.urdf (robot description, URDF)
Before this commit: robot project_model, 7 links, 6 joints
Joints:
- joint Joint_Vakuumgreifer: limit (none) -> lower=-3 upper=3 effort=100.0 velocity=0.1; type continuous -> revolute
